File: PCB/PSU/PSU.kicad_pcb (KiCad board)
At the start: 4 copper layers, 72.3 x 45 mm, 258 parts, among them J1 Backllight_Connector, J2 PSU_Jack, J3 PSU_Connector_Receptor, Q1 R4C, Q10 103 5G, Q11 6LS, Q12 Q, Q13 8LR, Q14 6LS, Q15 8LR, Q16 M2P, Q17 M2P, Q18 Q, Q19 M2P, Q2 K, Q20 W6, Q21 8C, Q22 8C, Q23 8C, Q24 6LS, Q25 8LB, Q26 G16, Q27 8C, Q28 W6, Q29 H15, Q3 6LS, Q30 8C, Q31 W6, Q32 K, Q33 8LR, Q34 6LS, Q35 8C, Q36 3P4J, Q37 8LR, Q4 8LR, Q5 8C, Q6 6LS, Q7 6LS, Q8 303 5H, Q9 KD 3.E, SW1 PSU-SW1, U1 D9D, U10 9742, U11 7W14, U12 J421, U13 J421, U2 TA, U3 6.5 5F, U4 MAX786CAI, U5 K2337, U6 7064, U7 5W01, U8 2556, U9 2556

Commit message: cleanup psu schematics
Parts:
- removed the R87 at (167.0, 116.7)
- C1: renamed from R97; value DNP -> ~
- C10: renamed from C12; value 1.2uF -> 1u
- C11: renamed from C3; value 5.2uF -> 4.7u
- C12: renamed from C39; value 10nF -> 0.01u
- C13: renamed from C1; value 150nF -> 0.1u
- C14: renamed from C52; value 1nF -> 1000p
- C15: renamed from C43; value 10pF -> 4.7p
- C16: renamed from C20; value 100pF -> 47p
- C17: renamed from C25; value 1.2nF -> 1000p
- C18: renamed from C21; value 12nF -> 0.01u
- C19: renamed from C46; value 150nF -> 0.1u
- C2: renamed from C29; value 10nF -> 0.01u
- C20: renamed from C27; value 1.2nF -> 1000p
- C21: renamed from C35; value 1.2nF -> 1000p
- C22: renamed from C37; value 180nF -> 0.1u
- C23: renamed from R91; value DNP -> ~
- C24: renamed from C49; value 180nF -> 0.1u
- C25: renamed from C44; value 180nF -> 0.1u
- C26: renamed from C28; value 150nF -> 0.1u
- C27: renamed from C36; value 150nF -> 0.1u
- C28: renamed from C31; value 1.2nF -> 1000p
- C29: renamed from C34; value 1.5uF -> 1u
- C3: renamed from C30; value 10nF -> 4700p
- C30: renamed from C33; value 24nF -> 0.022u
- C31: renamed from C13; value 1.5uF -> 1u
- C32: renamed from C14; value 1.5uF -> 1u
- C33: renamed from C47; value 150nF -> 0.1u
- C34: renamed from C55; value 1.5uF -> 1u
- C35: renamed from C38; value 1.5uF -> 1u
- C36: renamed from C23; value 1.5uF -> 1u
- C37: renamed from C40; value 10nF -> 0.01u
- C38: renamed from C19; value 18nF -> 0.1u
- C39: renamed from C26; value 10nF -> 0.01u
- C4: renamed from R95; value DNP -> ~
- C40: renamed from C22; value 10nF -> 0.01u
- C41: renamed from C48; value 10nF -> 0.01u
- C42: renamed from C18; value 120nF -> 0.1u
- C43: renamed from C64; value 120nF -> 0.1u
- C44: renamed from C58; value 1.5uF -> 1u
- C45: renamed from C59; value 150nF -> 0.1u
- C46: renamed from C41; value 1.5uF -> 1u
- C47: renamed from C60; value 1nF -> 1000p
- C48: renamed from C4; value 2.5nF -> 2200p
- C49: renamed from C65; value 100nF -> 0.1u
- C5: renamed from C42; value 120nF -> 0.1u
- C50: renamed from C17; value 10nF -> 0.01u
- C51: renamed from C32; value 10nF -> 0.01u
- C52: renamed from C66; value 1.2nF -> 1000p
- C53: renamed from C63; value 5.1nF -> 4700p
- C54: renamed from C7; value 150nF -> 0.1u
- C55: renamed from C9; value 10nF -> 0.01u
- C56: renamed from C10; value 3.6nF -> 3300p
- C57: renamed from C15; value 180nF -> 0.1u
- C58: renamed from C11; value 180nF -> 0.1u
- C59: renamed from C6; value 100pF -> 100p
- C6: renamed from C53; value 120nF -> 0.1u
- C60: renamed from C2; value 4.7nF -> 4700p
- C61: renamed from R1; value DNP -> ~
- C62: renamed from C5; value 150nF -> 0.1u
- C63: renamed from C8; value 24nF -> 0.022u
- C64: renamed from C62; value 100nF -> 0.1u
- C65: renamed from C24; value 150nF -> 0.1u
- C7: renamed from C51; value 120nF -> 0.1u
- C8: renamed from R66; value DNP -> ~
- C9: renamed from C16; value 150nF -> 0.1u
- CN1: renamed from J2; value PSU_Jack -> HEC3150-012120
- CN3: renamed from J3; value PSU_Connector_Receptor -> 179029-1
- CN4: renamed from J1; value Backllight_Connector -> DF13- 4P-1.25V
- D1: renamed from D7; value s.3 4F -> EC10QS03L
- D10: renamed from Q20; value W6 -> MA741WA
- D105: renamed from D6; value DNP -> EC11FS2
- D11: renamed from D5; value 3^9 -> MAZ8039-H
- D2: renamed from D8; value s.3 4F -> EC10QS03L
- D3: renamed from Q31; value W6 -> DCG010
- D4: renamed from Q2; value K -> SB007W03Q
- D5: renamed from Q19; value M2P -> MA741WA
- D50: renamed from Q12; value Q -> SB05-03Q
- D6: renamed from Q16; value M2P -> MA741WA
- D7: renamed from Q28; value W6 -> DCG010
- D8: renamed from Q32; value K -> SB007W03Q
- D9: renamed from Q17; value M2P -> MA741WA
- EC1: renamed from C50; value 56uF 25V EC -> 56u
- EC2: renamed from C45; value 33uF 20V -> 33u
- EC30: renamed from C54; value 47uF 6.3v -> 47u
- EC50: renamed from C61; value 47uF 6.3v -> 47u
- EC51: renamed from C56; value 47uF 6.3V -> 47u
- EC70: renamed from C57; value 15uF 16V -> 15u
- EC80: renamed from C67; value 18uF 50V -> 18u
- F4: renamed from F3; value 15 -> CCP2E15
- F5: renamed from F4; value 10 -> CCP2E10
- F6: renamed from F2; value 830mA -> 630mA
- L30: renamed from L2; value 10uH -> 22u
- L50: renamed from L5; value 10uH -> 10u
- L70: renamed from L3; value 68uH -> 68u
- L80: renamed from L4; value 470uH -> 470u
- L81: renamed from L1; value 10uH -> 10u
- Q1: renamed from Q36; value 3P4J -> 3P4J-ZK
- Q10: renamed from Q22; value 8C -> UN9213
- Q11: renamed from Q35; value 8C -> UN9213
- Q12: renamed from Q4; value 8LR -> UN9210-R
- Q123: renamed from Q8; value 303 5H -> FP303
- Q124: renamed from Q10; value 103 5G -> FP301
- Q13: renamed from Q5; value 8C -> UN9213
- Q14: renamed from Q34; value 6LS -> UN9110-S
- Q15: renamed from Q33; value 8LR -> UN9210-R
- Q16: renamed from Q37; value 8LR -> UN9210-R
- Q17: renamed from Q14; value 6LS -> UN9110-S
- Q18: renamed from Q21; value 8C -> UN9213
- Q19: renamed from Q15; value 8LR -> UN9210-R
- Q2: renamed from U13; value J421 -> 2SJ421
- Q20: renamed from Q30; value 8C -> UN9213
- Q21: renamed from U3; value 6.5 5F -> XN4609
- Q22: renamed from Q29; value H15 -> 2SJ204
- Q23: renamed from Q26; value G16 -> 2SK1590
- Q24: renamed from Q27; value 8C -> UN9213
- Q25: renamed from Q7; value 6LS -> UN9110-S
- Q26: renamed from Q6; value 6LS -> UN9110-S
- Q3: renamed from Q23; value 8C -> UN9213
- Q30: renamed from Q18; value Q -> SB05-03Q
- Q4: renamed from Q24; value 6LS -> UN9110-S
- Q5: renamed from Q25; value 8LB -> UN9210-R
- Q50: renamed from U9; value 2556 -> 2SK2556
- Q51: renamed from U8; value 2556 -> 2SK2556
- Q6: renamed from Q13; value 8LR -> UN9210-R
- Q7: renamed from Q11; value 6LS -> UN9110-S
- Q8: renamed from U12; value J421 -> 2SJ421
- Q9: renamed from Q3; value 6LS -> UN9110-S
- R111: renamed from R82; value DNP -> ~
- R26: renamed from R8; value 0.1 -> 100m
- R27: renamed from R7; value 0.1 -> 100m
- R3: renamed from R96; value 1.8k -> 1k
- R50: renamed from R55; value 1M -> 10M
- R55: renamed from R65; value 1k -> 100k
- R57: renamed from R50; value DNP -> ~
- R59: renamed from R85; value 10k -> 1k
- R66: renamed from R46; value 1M -> 10M
- R72: renamed from R40; value 0.22 -> 220m
- R73: renamed from R32; value 0.1 -> 100m
- R77: renamed from R108; value DNP -> ~
- R79: renamed from R23; value 0.1 -> 100m
- R80: renamed from R25; value 0.1 -> 100m
- R81: renamed from R34; value 0.1 -> 100m
- R88: renamed from R115; value 11K -> 11k
- RT1: renamed from R29; value 103 (RT2) -> 103HT-xx
- RT2: renamed from R26; value 103 (RT1) -> 103HT-xx
- SW1: value PSU-SW1 -> ~
- U1: value D9D -> S-80745SN-D9-X
- U100: renamed from U6; value 7064 -> NJU7064V
- U101: renamed from U2; value TA -> TA75S393F
- U102: renamed from U7; value 5W01 -> TA75W01FU
- U103: renamed from U11; value 7W14 -> TC7W14FK
- U2: renamed from Q9; value KD 3.E -> S-81350HG
- U4: renamed from U10; value 9742 -> BA9742
- U5: renamed from Q1; value R4C -> LM4040CIM3-4.1
- Z1: renamed from D4; value 18 -> MAZ8180-M
- Z3: renamed from D2; value 5-9 -> MAZ8056-M
- Z4: renamed from D3; value DNP -> ~
- Z5: renamed from D1; value 8-2 -> MAZ8082-M
- moved EC70 2.54 mm to (120.0, 99.0), turned to 180 degrees
- moved EC30 2.50 mm to (144.0, 109.2), turned to 180 degrees
- moved EC50 2.50 mm to (137.2, 109.2), turned to 180 degrees
- turned Z4 to 180 degrees
- renumbered F5 to F2, R99 to R1, R70 to R10, R116 to R100, R4 to R101, R11 to R102, R35 to R103, R19 to R104, R18 to R105, R10 to R106, R93 to R107, R94 to R108, R27 to R109, R78 to R11, R58 to R110, R77 to R12, R53 to R13, R54 to R14, R22 to R15, R28 to R16, R21 to R17, R31 to R18, R30 to R19, R98 to R2, R5 to R20, R73 to R21, R92 to R22, R2 to R23, R3 to R24, R6 to R25, R64 to R28, R52 to R29, R69 to R30, R101 to R31, R49 to R32, R102 to R33, R105 to R34, R57 to R35, R90 to R36, R63 to R38, R44 to R39, R76 to R4, R45 to R40, R62 to R41, R112 to R43, R107 to R44, R106 to R45, R67 to R46, R103 to R47, R109 to R48, R113 to R49, R111 to R5, R68 to R51, R59 to R52, R51 to R53, R47 to R54, R60 to R56, R84 to R58, R75 to R6, R61 to R60, R41 to R61, R39 to R62, R89 to R63, R88 to R64, R83 to R65, R36 to R67, R86 to R68, R80 to R69, R71 to R7, R104 to R70, R48 to R71, R56 to R74, R43 to R75, R110 to R76, R100 to R78, R72 to R8, R118 to R82, R114 to R83, R20 to R84, R12 to R85, R24 to R86, R81 to R87, R117 to R89, R74 to R9, R13 to R90, R33 to R91, R14 to R92, R9 to R93, R79 to R94, R15 to R95, R17 to R96, R38 to R97, R37 to R98, R16 to R99, U4 to U3, U5 to U30
Connections:
- net BATT_POS renamed Net-(CN5-Pad2)
- net C1_1 renamed Net-(C60-Pad1)
- net C1_2 renamed Net-(U4-FB2)
- net C31_1 renamed Net-(Q24-C)
- net C32_1 renamed Net-(Q24-B)
- net C33_1 renamed Net-(Q23-G)
- net C35_2 renamed Net-(Q22-D)
- net C36_1 renamed Net-(Q21A-Q1_B)
- net C36_2 renamed Net-(Q20-C)
- net C6_1 renamed Net-(C48-Pad1)
- net C6_2 renamed Net-(U103C-3Y)
- net C8_1 renamed Net-(U4-DT1)
- net D18_2_3_PC110 renamed LCD_BKLIT_INVEN
- net D1_2 renamed Net-(Q13-B)
- net D2_3_PC110 renamed VIN_AC_DETECT
- net F2_1 renamed Net-(CN5-Pad1)
- net F3_1 renamed Net-(C57-Pad1)
- net F65_ENAVEE_PC110 renamed VAA_LCD_ENABLE
- net J1_4 renamed Net-(C65-Pad2)
- net J5_33_PC110 renamed EXT_DEV_DETSW
- net J5_6_PC110 renamed CHG_SUBPWR
- net JRC_IN1+ renamed Net-(U100A-1IN+)
- net JRC_IN1- renamed Net-(U100A-1IN-)
- net JRC_IN2+ renamed Net-(U100B-2IN+)
- net JRC_IN2- renamed Net-(U100B-2IN-)
- net JRC_IN3+ renamed Net-(U100C-3IN+)
- net JRC_IN3- renamed Net-(D5-C2)
- net JRC_IN4+ renamed Net-(D5-C1)
- net JRC_IN4- renamed Net-(U100D-4IN-)
- net JRC_VDD renamed +5V_CHGMON
- net L1_2 renamed Net-(D105-C)
- net L2_2 renamed Net-(Q124A-C)
- net M38_P20_PC110 renamed CHG_CONT_1
- net M38_P21_PC110 renamed CHG_CONT_2
- net M38_P52_PC110 renamed CHG_MONPWR_EN
- net M38_P53_PC110 renamed MONT_VOLT_ENABLE
- net M38_P60_PC110 renamed BAT_MON_DISCHGCURR
- net M38_P61_PC110 renamed BAT_MON_CHGCURR
- net M38_P63_PC110 renamed BAT_MONT_VOLT
- net M38_P64_PC110 renamed VIN_AC_MON_VOLT
- net M38_VREF_PC110 renamed VREF
- net MAX_BST3 renamed Net-(D9-C2)
- net MAX_BST5 renamed Net-(D9-C1)
- net MAX_CS3 renamed Net-(U3-CS3)
- net MAX_CS5 renamed Net-(U3-CS5)
- net MAX_DH3 renamed Net-(U3-DH3)
- net MAX_DH5 renamed Net-(Q50-G)
- net MAX_DL3 renamed Net-(U3-DL3)
- net MAX_DL5 renamed Net-(Q51-G)
- net MAX_FB3 renamed Net-(U3-FB3)
- net MAX_LX3 renamed Net-(Q30-C)
- net MAX_LX5 renamed Net-(D50-C)
- net MAX_REF renamed Net-(U3-REF)
- net MAX_SS3 renamed Net-(U3-SS3)
- net MAX_SS5 renamed Net-(U3-SS5)
- net MAX_VL renamed +5V_MAX786_VL
- net MAX_VL+ renamed Net-(U3-V+)
- net ON3_ON5_VH_SHDN# renamed Net-(U3-ON3)
- net PNET4_PC110 renamed VSYS
- net PWR_IN_10v5 renamed VIN_AC
- net PWR_IN_NEG renamed Net-(C1-Pad2)
- net PWR_IN_POS renamed Net-(CN1-Pad1)
- net PWR_IN_POS_Fuse renamed Net-(C1-Pad1)
- net Q13_3 renamed Net-(Q6-C)
- net Q14_2 renamed Net-(D10-A)
- net Q20_1 renamed Net-(D6-C1)
- net Q22_1 renamed Net-(Q4-B)
- net Q27_3 renamed Net-(Q22-G)
- net Q29_2 renamed MONT_V_EN_OR
- net Q30_2 renamed CHG_CONT_2_OR
- net Q33_2 renamed VBAT
- net Q33_3 renamed Net-(Q14-C)
- net Q36_3 renamed Net-(Q16-C)
- net Q3_1 renamed Net-(Q12-B)
- net Q3_3 renamed Net-(Q10-C)
- net Q43_2_PC110 renamed VAA_LCD
- net Q49_1_PC110 renamed TEMPSENS
- net Q4_1 renamed Net-(Q9-B)
- net Q6_2 renamed VREF_BA9742
- net Q7_1 renamed Net-(Q26-B)
- net Q7_3 renamed Net-(Q26-C)
- net Q8_1 renamed Net-(Q123A-B)
- net Q8_5 renamed Net-(Q123A-C)
- net Q9_1 renamed Net-(Q124A-B)
- net R104_1 renamed Net-(U102B-2IN+)
- net R106_1 renamed Net-(C7-Pad2)
- net R106_2 renamed Net-(C6-Pad1)
- net R111_! renamed Net-(U102A-1IN+)
- net R111_2 renamed Net-(Q17-C)
- net R115_2 renamed Net-(C52-Pad2)
- net R11_1 renamed Net-(U103C-3A)
- net R17_2 renamed Net-(Q25-B)
- net R19_1 renamed Net-(U103A-1A)
- net R20_1 renamed Net-(U4-DT2)
- net R21_1 renamed Net-(Q6-B)
- net R21_2 renamed Net-(U1-OUT)
- net R24_2 renamed Net-(U103A-1Y)
- net R26_2 renamed Net-(R16-Pad2)
- net R284_2_PC110 renamed VSW
- net R284_2_PC110_Fuse renamed Net-(C49-Pad1)
- net R2_2 renamed Net-(D4-A1)
- net R31_1 renamed Net-(U1-VDD)
- net R32_1 renamed Net-(U4-INV2)
- net R35_2 renamed Net-(Q7-B)
- net R36_1 renamed Net-(U4-INV1)
- net R36_2 renamed Net-(C56-Pad2)
- net R38_1 renamed Net-(D10-C2)
- net R412_1_PC110 renamed LCD_BKLIT_ADJ
- net R48_2 renamed Net-(D10-C1)
- net R50_1 renamed Net-(Q20-E)
- net R50_2 renamed Net-(U101A-1IN+)
- net R51_1 renamed Net-(D6-A)
- net R51_2 renamed Net-(Q19-E)
- net R54_2 renamed Net-(R61-Pad2)
- net R56_1 renamed Net-(C39-Pad1)
- net R59_1 renamed Net-(Q18-B)
- net R61_1 renamed Net-(Q19-B)
- net R68_1 renamed Net-(Q17-B)
- net R68_2 renamed Net-(Q18-C)
- net R6_2 renamed Net-(D4-C)
- net R70_2 renamed Net-(Q5-C)
- net R72_1 renamed Net-(Z1-A)
- net R72_2 renamed Net-(Q1-G)
- net R73_2 renamed Net-(Q5-B)
- net R73_2_PC110 renamed VAA_LCD_ADJ
- net R76_1 renamed Net-(R6-Pad1)
- net R77_1 renamed AC_IN_DETECT_DIV
- net R77_2 renamed Net-(Q10-B)
- net R78_2 renamed Net-(Q4-C)
- net R80_1 renamed Net-(Q25-C)
- net R82_1 renamed Net-(Q20-B)
- net R89_1 renamed Net-(R63-Pad1)
- net R91_1 renamed Net-(Q15-C)
- net R91_2 renamed Net-(Q14-B)
- net R92_2 renamed Net-(Q11-B)
- net SW1_2 renamed Net-(R107-Pad1)
- net U11_1 renamed BA9742_CT
- net U11_15 renamed Net-(U4-SCP)
- net U11_2 renamed Net-(U4-RT)
- net U11_5 renamed Net-(U4-FB1)
- net U11_9 renamed Net-(U4-VCC)
- net U21_131_PC110 renamed +12V_ENABLE
- net U3_1 renamed Net-(Q2-G)
- net U3_6 renamed Net-(D8-C)
- net U54_1D_PC110 renamed VSW_ENABLE_1
- net U54_1Q_PC110 renamed VSW_ENABLE_2
- net U54_VCC_PC110 renamed +5V_STBY
- net U6_2 renamed Net-(U102A-1IN-)
- net U6_6 renamed Net-(U102B-2IN-)
- net U6_7 renamed Net-(D6-C2)
- C10 pad 2: C14_2 -> Net-(Q7-C)
- C26 pad 2: PNET5_PC110 -> +5V_SW
- C40 pad 1: PNET1_PC110 -> +3V3
- C58 pad 1: D28_1_PC110 -> +12V
- C59 pad 2: D28_1_PC110 -> +12V
- C64 pad 2: PNET5_PC110 -> +5V_SW
- CN3 pad 10: PNET5_PC110 -> +5V_SW
- CN3 pad 11: PNET5_PC110 -> +5V_SW
- CN3 pad 12: D28_1_PC110 -> +12V
- CN3 pad 28: PNET1_PC110 -> +3V3
- CN3 pad 31: PNET5_PC110 -> +5V_SW
- CN3 pad 8: PNET1_PC110 -> +3V3
- CN4 pad MP: J1_MP2 -> (no net)
- D4 pad 3: PNET5_PC110 -> +5V_SW
- EC30 pad 1: PNET1_PC110 -> GND
- EC30 pad 2: GND -> +3V3
- EC50 pad 1: PNET5_PC110 -> GND
- EC50 pad 2: GND -> +5V_SW
- EC51 pad 2: PNET5_PC110 -> +5V_SW
- EC70 pad 1: D28_1_PC110 -> GND
- EC70 pad 2: GND -> +12V
- Q124 pad 4: D28_1_PC110 -> +12V
- Q15 pad 1: R88_1 -> Net-(Q15-B)
- Q19 pad 3: PNET5_PC110 -> +5V_SW
- Q7 pad 3: C14_2 -> Net-(Q7-C)
- R58 pad 2: PNET5_PC110 -> +5V_SW
- R72 pad 1: PNET1_PC110 -> +3V3
- R73 pad 1: PNET1_PC110 -> +3V3
- R75 pad 1: PNET1_PC110 -> +3V3
- R79 pad 1: PNET5_PC110 -> +5V_SW
- R80 pad 1: PNET5_PC110 -> +5V_SW
- R81 pad 1: PNET5_PC110 -> +5V_SW
- R82 pad 1: PNET5_PC110 -> +5V_SW
- R84 pad 2: PNET5_PC110 -> +5V_SW
- R96 pad 2: PNET5_PC110 -> +5V_SW
- R99 pad 2: D28_1_PC110 -> +12V
- RT1 pad 2: PNET5_PC110 -> +5V_SW
- RT2 pad 1: PNET5_PC110 -> +5V_SW
- SW1 pad 3: SW1_3 -> (no net)
- SW1 pad 4: SW1_4 -> (no net)
- U1 pad 4: U1_4 -> (no net)
- U1 pad 5: U1_5 -> (no net)
- U101 pad 5: PNET5_PC110 -> +5V_SW
- U103 pad 8: PNET5_PC110 -> +5V_SW
- U2 pad 3: C14_2 -> Net-(Q7-C)
- U3 pad 21: PNET5_PC110 -> +5V_SW
- U3 pad 7: MAX_Q2 -> unconnected-(U3-Q2-Pad7)
- U3 pad 8: MAX_Q1 -> unconnected-(U3-Q1-Pad8)
- U5 pad 2: Q1_2 -> (no net)
- Z4 pad 1: GND -> Net-(Q7-C)
- Z4 pad 2: C14_2 -> GND
Routing:
- net PNET5_PC110: track 168.9 -> 0.00 mm, vias 9 -> 0
- net +5V_SW: track 0.00 -> 168.9 mm, vias 0 -> 9
- net D28_1_PC110: track 36.6 -> 0.00 mm
- net +12V: track 0.00 -> 36.6 mm
- net PNET1_PC110: track 20.4 -> 0.00 mm
- net +3V3: track 0.00 -> 20.4 mm
- net Net-(Q7-C): track 0.00 -> 11.0 mm
- net C14_2: track 11.0 -> 0.00 mm
- net R88_1: track 1.33 -> 0.00 mm
- net Net-(Q15-B): track 0.00 -> 1.33 mm
- added copper zone on F.Cu, net +3V3
- added copper zone on B.Cu, net +5V_SW
- added copper zone on In1.Cu, net +5V_SW
- added copper zone on B.Cu, net CHG_CONT_2
- added copper zone on F.Cu, net Net-(Q18-C)
- removed copper zone on In1.Cu, net (none)
- removed copper zone on F.Cu, net Net-(Q30-C)
- removed copper zone on B.Cu, net PNET1_PC110
- removed copper zone on F.Cu, net PNET1_PC110
- removed copper zone on B.Cu, net PNET5_PC110
- removed copper zone on In1.Cu, net PNET5_PC110
