File: PCB/DockingStation/DockingStation.kicad_sch (KiCad schematic)
At the start: 252 parts, among them CN1 DSUB-15-HD_Socket_Horizontal_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, CN2 FDC_Connector, CN4 DSUB-25_Socket_Horizontal_P2.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, CN5 DSUB-9_Pins_Horizontal_P2.77x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, CN6 PS2 Connector, CN7 PS2 Connector, CN8 BarrelJack_Horizontal_PC110, J1 25-1MP_P0.5mm_Horizontal, J2 25-1MP_P0.5mm_Horizontal, J3 25-1MP_P0.5mm_Horizontal, J4 25-1MP_P0.5mm_Horizontal, Q1 3P4J, Q2 8C, U1 74VHCT244, U2 DNP (LT1237CS), U3 DS14C535MSA, U4 DNP

Commit message: cleaned up dock board schematics
Parts:
- removed C1: 330nF, Capacitor_SMD:C_0805_2012Metric, symbol PCM_Elektuur:C
- removed C10: 1nF, Capacitor_SMD:C_0603_1608Metric, symbol PCM_Elektuur:C
- removed C11: 2.5uF, Capacitor_SMD:C_1206_3216Metric, symbol PCM_Elektuur:C
- removed C12, C15, C17, C19, C21, C23, C25, C27, C29, C31, C32, C34, C35, C9: 280nF, Capacitor_SMD:C_0603_1608Metric, symbol PCM_Elektuur:C
- removed C13, C14, C16, C18, C20, C22, C24, C26, C28, C30: 82pF, Capacitor_SMD:C_0603_1608Metric, symbol PCM_Elektuur:C
- removed C2: 1nF, Capacitor_SMD:C_0805_2012Metric, symbol PCM_Elektuur:C
- removed C3, C4: 200pF, Capacitor_SMD:C_0805_2012Metric, symbol PCM_Elektuur:C
- removed C33: 330nF, Capacitor_SMD:C_0603_1608Metric, symbol PCM_Elektuur:C
- removed C37, C38, C39, C40, C41, C42, C43, C44, C63, C64, C65, C66: 200pF, Capacitor_SMD:C_0603_1608Metric, symbol PCM_Elektuur:C
- removed C45, C46, C47, C48, C49, C50, C51, C52, C53, C54, C55, C56, C57, C58, C59, C60, C61: 200nF, Capacitor_SMD:C_0603_1608Metric, symbol PCM_Elektuur:C
- removed C62, C67, C78: 250nF, Capacitor_SMD:C_0603_1608Metric, symbol PCM_Elektuur:C
- removed C68, C73, C74, C83: DNP, Capacitor_SMD:C_0603_1608Metric, symbol PCM_Elektuur:C
- removed C69, C71: DNP, Capacitor_SMD:C_1206_3216Metric, symbol PCM_Elektuur:C
- removed C70, C72: DNP, Capacitor_SMD:C_0805_2012Metric, symbol PCM_Elektuur:C
- removed C75: 150nF, Capacitor_SMD:C_0603_1608Metric, symbol PCM_Elektuur:C
- removed C76, C77: 10nF, Capacitor_SMD:C_0603_1608Metric, symbol PCM_Elektuur:C
- removed C79, C80, C81, C82: 360nF, Capacitor_SMD:C_0805_2012Metric, symbol PCM_Elektuur:C
- removed CN1: DSUB-15-HD_Socket_Horizontal_P2.29x1.90mm_EdgePin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, Connector_Dsub:DSUB-15-HD_Socket_Horizontal_P2.29x1.90mm_EdgePinOffset3.03mm_Housed_MountingHolesOffset4.94mm, symbol Connector:DE15_Pins_HighDensity
- removed CN2: FDC_Connector, DockingStation:FDC_Connector, symbol Connector_Generic:Conn_01x26
- removed CN4: DSUB-25_Socket_Horizontal_P2.77x2.84mm_EdgePinOff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, Connector_Dsub:DSUB-25_Socket_Horizontal_P2.77x2.84mm_EdgePinOffset4.94mm_Housed_MountingHolesOffset4.94mm, symbol Connector:DB25_Socket
- removed CN5: DSUB-9_Pins_Horizontal_P2.77x2.84mm_EdgePinOffset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, Connector_Dsub:DSUB-9_Pins_Horizontal_P2.77x2.84mm_EdgePinOffset4.94mm_Housed_MountingHolesOffset4.94mm, symbol Connector:DE9_Socket
- removed CN6, CN7: PS2 Connector, DockingStation:PS2 Connector, symbol Connector:Mini-DIN-6
- removed CN8: BarrelJack_Horizontal_PC110, DockingStation:BarrelJack_Horizontal_PC110, symbol Connector:Barrel_Jack
- removed D2, D3: s.3 5J, Diode_SMD:D_2010_5025Metric, symbol Device:D_Schottky
- removed DA1, DA10, DA2, DA3, DA4, DA6, DA7, DA8: 1W, Package_TO_SOT_SMD:SOT-323_SC-70, symbol Device:D_Dual_Series_KAC
- removed DA11, DA12: DNP, Package_TO_SOT_SMD:SOT-23W, symbol Device:D_Dual_CommonCathode_AAK_Parallel
- removed DA9: SOT-323_SC-70, Package_TO_SOT_SMD:SOT-323_SC-70, symbol Device:D_Dual_Series_KAC
- removed F1: 50v x1G0 JX30, Fuse:Fuse_Littelfuse_395Series, symbol PCM_Elektuur:F
- removed J1, J2, J3, J4: 25-1MP_P0.5mm_Horizontal, DockingStation:25-1MP_P0.5mm_Horizontal_PC110_dock, symbol Connector_Generic:Conn_01x25
- removed L1, L2, L3, L34, L37, L38: 300nH, Inductor_SMD:L_0805_2012Metric, symbol PCM_Elektuur:L
- removed L11, L13, L14, L15, L16, L17, L18, L19, L20, L21, L22, L23, L24, L25, L26, L27, L28, L29, L30, L31, L39, L40, L41, L42, L43, L44, L45, L46, L47, L48, L49, L5, L50, L51, L52, L53, L54, L55, L56, L57, L58, L59, L6, L60, L61, L62, L63, L64, L65, L66, L67: 680nH, Inductor_SMD:L_0805_2012Metric, symbol PCM_Elektuur:L
- removed L68: EMI_Transformer, DockingStation:EMI_Transformer, symbol Device:Filter_EMI_CommonMode
- removed Q1: 3P4J, Package_TO_SOT_SMD:TO-252-2, symbol PCM_Elektuur:Th
- removed Q2: 8C, Package_TO_SOT_SMD:SOT-323_SC-70, symbol PCM_Transistor_BJT_AKL:Q_NPN_Generic_BEC
- removed R1, R2: 33, Resistor_SMD:R_0805_2012Metric, symbol PCM_Elektuur:R
- removed R10, R11, R29, R40, R42, R43, R44, R45, R46, R47, R48, R49, R50, R51, R60, R61, R62, R63, R64, R65, R66, R67: DNP, Resistor_SMD:R_0603_1608Metric, symbol PCM_Elektuur:R
- removed R12, R13, R14, R15, R16, R17, R18, R19, R20, R21, R22, R23, R24, R25, R26, R27, R28: 10, Resistor_SMD:R_0603_1608Metric, symbol PCM_Elektuur:R
- removed R3, R4: 33, Resistor_SMD:R_0603_1608Metric, symbol PCM_Elektuur:R
- removed R30, R31, R32, R33, R34, R35, R36, R37: 1k, Resistor_SMD:R_0805_2012Metric, symbol PCM_Elektuur:R
- removed R38: 0, Resistor_SMD:R_0805_2012Metric, symbol PCM_Elektuur:R
- removed R39, R41, R5, R52, R53, R54, R55, R56, R57, R58, R59, R68, R69, R7, R70, R71, R72, R73, R74, R75, R8: 0, Resistor_SMD:R_0603_1608Metric, symbol PCM_Elektuur:R
- removed R6, R9: 470k, Resistor_SMD:R_0603_1608Metric, symbol PCM_Elektuur:R
- removed RA2, RA3, RA4: 47k, Resistor_SMD:R_Array_Concave_4x0603, symbol Device:R_Pack04
- removed RA5, RA6: 470k, Resistor_SMD:R_Array_Concave_4x0603, symbol Device:R_Pack04
- removed RA7, RA8: DNP, Resistor_SMD:R_Array_Concave_4x0603, symbol Device:R_Pack04
- removed SSFC1: Fuse_2010_5025Metric, Fuse:Fuse_2010_5025Metric, symbol PCM_Elektuur:F
- removed U1: 74VHCT244, Package_SO:SSOP-20_4.4x6.5mm_P0.65mm, symbol 74xx:74HCT244
- removed U2: DNP (LT1237CS), Package_SO:SSOP-28_5.3x10.2mm_P0.65mm, symbol DockingStation:LT1237
- removed U3: DS14C535MSA, Package_SO:SSOP-28_5.3x10.2mm_P0.65mm, symbol DockingStation:DS14C535MSA
- removed U4: DNP, Package_TO_SOT_SMD:SOT-23-5, symbol 74xGxx:74AHC1G14
- removed ZD1: 18-, Diode_SMD:D_0805_2012Metric, symbol Diode:ZPDxx
- removed ZD4: 5_1, Diode_SMD:D_0805_2012Metric, symbol Diode:ZPDxx
- added C31, C32, C33, C34, C35, C36: 0.22u, symbol DockingStation:C
- added J1, J2: 086212025340800, symbol DockingStation:CN_25+PAD
- added J3, J4: 086210025340800, symbol DockingStation:CN_25+PAD
- added R7, R8: 0, symbol DockingStation:R
Connections:
- net GND: now also C31.1, C32.2, C33.2, C34.1, C35.1, C36.1, J1.1, J1.10, J1.12, J1.25, J1.6, J1.8, J2.1, J2.16, J3.1, J4.25, R7.2, R8.2
- net VGA_BLUE: now also J1.11
- net VGA_GREEN: now also J1.9
- net VGA_RED: now also J1.7
- new net: J3.2, R7.1
- new net: J2.2, R8.1
- new net +5V_232: C36.2, J4.15
- new net +5V_FDD: C34.2, C35.2, J2.12, J2.13, J3.13
- new net +5V_PS2: C31.2, J3.16
- new net +5V_VGA: C32.1, C33.1, J2.21, J3.21
- new net 1284_BUSY: J3.22
- new net 1284_D1: J4.5
- new net 1284_D2: J4.4
- new net 1284_D3: J4.3
- new net 1284_D4: J4.2
- new net 1284_D5: J4.1
- new net 1284_D6: J3.25
- new net 1284_D7: J2.25
- new net 1284_D8: J3.24
- new net 1284_PERROR: J2.23
- new net 1284_SELECT: J3.23
- new net 1284_~{ACK}: J1.5
- new net 1284_~{AUTOFD}: J1.3
- new net 1284_~{FAULT}: J2.24
- new net 1284_~{INIT}: J1.4
- new net 1284_~{SELECTIN}: J1.2
- new net 1284_~{STROBE}: J4.6
- new net 232_CTS: J2.19
- new net 232_DCD: J3.17
- new net 232_DSR: J2.17
- new net 232_DTR: J3.20
- new net 232_EN: J2.22
- new net 232_RI: J2.20
- new net 232_RTS: J2.18
- new net 232_RXD: J3.18
- new net 232_TXD: J3.19
- new net FDD_DETFDD: J2.11
- new net FDD_DIRSEL: J3.7
- new net FDD_DISKCHG: J3.12
- new net FDD_DRATE0: J2.5
- new net FDD_DRATE1: J3.3
- new net FDD_DRVSEL: J3.5
- new net FDD_HEADSEL: J3.11
- new net FDD_INDEX: J3.4
- new net FDD_MOTON: J3.6
- new net FDD_PLUTO1: J2.3
- new net FDD_PLUTO2: J2.4
- new net FDD_PLUTO3: J2.6
- new net FDD_PLUTO4: J2.9
- new net FDD_RDATA: J2.10
- new net FDD_STEP: J2.7
- new net FDD_TRK00: J3.9
- new net FDD_WDATA: J3.8
- new net FDD_WGATE: J2.8
- new net FDD_WPRT: J3.10
- new net GND_VIN_AC: J1.19, J1.20, J1.21, J1.22, J1.23
- new net PS2_1_CLOCK: J3.15
- new net PS2_1_DATA: J3.14
- new net PS2_2_CLOCK: J2.15
- new net PS2_2_DATA: J2.14
- new net VGA_HSYNC: J4.11
- new net VGA_VSYNC: J4.8
- new net VIN_AC: J4.19, J4.20, J4.21, J4.22, J4.23
- new net VIN_AC_DET: J4.13, J4.14
- new net VIN_AC_DET_DIV: J1.15
- new net VIN_AC_LP: J1.13
- no-connect marks 29 -> 17
Other:
- added sheet AC Input (acinput.kicad_sch)
- added sheet FDD Port (fdd.kicad_sch)
- added sheet PS2 Port (ps2.kicad_sch)
- added sheet Parallel Port (parallel.kicad_sch)
- added sheet Serial Port (serial.kicad_sch)
- added sheet VGA (vga.kicad_sch)
- note added: "1"
- note added: "10"
- note added: "100"
- note added: "11"
- note added: "12"
- note added: "13"
- note added: "14"
- note added: "15"
- note added: "16"
- note added: "17"
- note added: "18"
- note added: "19"
- note added: "2"
- note added: "20"
- note added: "21"
- note added: "22"
- note added: "23"
- note added: "24"
- note added: "25"
- note added: "26"
- note added: "27"
- note added: "28"
- note added: "29"
- note added: "3"
- note added: "30"
- note added: "31"
- note added: "32"
- note added: "33"
- note added: "34"
- note added: "35"
- note added: "36"
- note added: "37"
- note added: "38"
- note added: "39"
- note added: "4"
- note added: "40"
- note added: "41"
- note added: "42"
- note added: "43"
- note added: "44"
- note added: "45"
- note added: "46"
- note added: "47"
- note added: "48"
- note added: "49"
- note added: "5"
- note added: "50"
- note added: "51"
- note added: "52"
- note added: "53"
- note added: "54"
- note added: "55"
- note added: "56"
- note added: "57"
- note added: "58"
- note added: "59"
- note added: "6"
- note added: "60"
- note added: "61"
- note added: "62"
- note added: "63"
- note added: "64"
- note added: "65"
- note added: "66"
- note added: "67"
- note added: "68"
- note added: "69"
- note added: "7"
- note added: "70"
- note added: "71"
- note added: "72"
- note added: "73"
- note added: "74"
- note added: "75"
- note added: "76"
- note added: "77"
- note added: "78"
- note added: "79"
- note added: "8"
- note added: "80"
- note added: "81"
- note added: "82"
- note added: "83"
- note added: "84"
- note added: "85"
- note added: "86"
- note added: "87"
- note added: "88"
- note added: "89"
- note added: "9"
- note added: "90"
- note added: "91"
- note added: "92"
- note added: "93"
- note added: "94"
- note added: "95"
- note added: "96"
- note added: "97"
- note added: "98"
- note added: "99"
- note added: "Dock connected via Flex Cable"
- company: Recreated by: Ahmad Byagowi -> (none)
- title: PC110 Docking Station -> P00-3E1263-02 : IBM PalmTop PC110 Docking Station board
