File: PCB/Modem/Modem.kicad_sch (KiCad schematic)
At the start: 90 parts, among them IC10 AT32, IC17 EA, IC2 EA, IC3 Line Module, IC7 EA, IC9 EA, Q3 123, Q4 CQ, T1 Iso Trans

Commit message: cleanup modem schematic
Parts:
- removed C1, C3, C4: 330nF, symbol PCM_Elektuur:C
- removed C30: 1.5uF, symbol PCM_Elektuur:C
- removed C31: 230nF, symbol PCM_Elektuur:C
- removed C32: 1.2uF, symbol PCM_Elektuur:C
- removed C45: 47uF, symbol PCM_Elektuur:C
- removed C5: 250nF, symbol PCM_Elektuur:C
- removed C59, C60, C62: 280nF, symbol PCM_Elektuur:C
- removed C70, C72: 1.8uF, symbol PCM_Elektuur:C
- removed C71: 1.3uF, symbol PCM_Elektuur:C
- removed C73: 100pF, symbol PCM_Elektuur:C
- removed C74: 220nF, symbol PCM_Elektuur:C
- removed CNP4: ~, symbol Modem:M_Conn
- removed D1, D7, D9: TO-269AA, Package_SO:TSSOP-4_4.4x5mm_P4mm, symbol Diode_Bridge:MDB6S
- removed D4: 5, symbol PCM_Elektuur:D
- removed DA1: M1T, symbol Device:D_Dual_CommonAnode_AKK_Split
- removed IC10: AT32, symbol 74xx:74LS32
- removed IC11: ~, symbol Modem:EN29F040A
- removed IC12: ~, symbol Modem:681000ALP
- removed IC17, IC2, IC7, IC9: EA, symbol 74xGxx:74AHC1G14
- removed IC3: Line Module, symbol Connector_Generic:Conn_01x18
- removed JCNP1: Tel Line, symbol Connector:4P4C
- removed L1, L2: 1.2uH, symbol PCM_Elektuur:L
- removed NF4: 4.5nH, symbol PCM_Elektuur:L
- removed PC2: TLS124, OptoDevice:Sharp_GP2S700HCP, symbol Sensor_Proximity:GP2S700HCP
- removed Q3: 123, symbol Simulation_SPICE:NPN
- removed Q4: CQ, symbol Simulation_SPICE:NPN
- removed R1: 12k, symbol PCM_Elektuur:R
- removed R10, R11: 38k, symbol PCM_Elektuur:R
- removed R100: 470k, symbol PCM_Elektuur:R
- removed R101, R102, R103, R104, R105, R106, R107, R108, R109, R110, R111, R112, R114, R115, R116, R117, R118, R119, R120, R121, R122, R123, R124, R125, R126, R127, R128, R129, R130, R131, R132, R98, R99: 100, symbol PCM_Elektuur:R
- removed R14: 560k, symbol PCM_Elektuur:R
- removed R16, R17, R18: 10k, symbol PCM_Elektuur:R
- removed R22, R23, R27: DNP, symbol PCM_Elektuur:R
- removed R52: 1k, symbol PCM_Elektuur:R
- removed R73: 120, symbol PCM_Elektuur:R
- removed R75: 2.2k, symbol PCM_Elektuur:R
- removed R76: 2.4k, symbol PCM_Elektuur:R
- removed R8: 22k, symbol PCM_Elektuur:R
- removed R81: 100k, symbol PCM_Elektuur:R
- removed T1: Iso Trans, Transformer_SMD:Transformer_ED8_4-Lead_10.5x8mm_P5mm, symbol Transformer:ED8_4
- removed VA1: R-nonlin, symbol PCM_Elektuur:R-nonlin
- added C2, C34: 1000p, symbol Modem:C
- added C23, C32, C70, C71, C72: 1u, symbol Modem:C
- added C24, C31, C58, C74: 0.22u, symbol Modem:C
- added C28: 10u, symbol Modem:C
- added C45: 47u, symbol Modem:C_POL
- added C46, C47, C48, C49: 0.022u, symbol Modem:C
- added C57: 8.2u, symbol Modem:C
- added C73: 100p, symbol Modem:C
- added CNP4: 8-176757-6, symbol Modem:CN_26
- added D5: RB715F, symbol Modem:D_CATHODE-COM
- added DA1: MA724, symbol Modem:D_2x
- added IC10: TC74ACT32FT, symbol Modem:74_OR
- added IC17: TC7S14FU, symbol Modem:74-1G_INV-SCHMITT
- added IC18: R3111N331C, symbol Modem:R3111
- added IC3: (no value), symbol Modem:CN_18
- added unit 3 of IC5
- added NF1, NF4: 330n, symbol Modem:L
- added NF2: 560n, symbol Modem:L
- added NF3: 0, symbol Modem:R
- added OSC1: 41.472MHz, symbol Modem:OSC
- added Q3: DTC143ZUA, symbol Modem:NPN
- added Q4: 2SC4097-Q, symbol Modem:NPN
- added R1, R8: 12k, symbol Modem:R
- added R10, R11: 39k, symbol Modem:R
- added R100, R51, R72, R79: 470k, symbol Modem:R
- added R133, R21, R47, R49, R67: 10k, symbol Modem:R
- added R16, R17, R19, R98, R99: 100, symbol Modem:R
- added R22, R23, R27: (no value), symbol Modem:R
- added R26, R33, R34: 10, symbol Modem:R
- added R3, R41, R43: 4.7k, symbol Modem:R
- added R35: 20, symbol Modem:R
- added R44: 51, symbol Modem:R
- added R48: 3.3, symbol Modem:R
- added R52: 1k, symbol Modem:R
- added R76: 2.4k, symbol Modem:R
- IC5: value ~ -> MN195001MFM-6
Connections:
- net AGND: now also C45.1 (2), C57.1, C71.2, C72.2, C73.1, C74.2, DA1.3 (C1), IC17.3 (GND), IC3.14, IC3.7, NF4.1, Q3.2 (E), R52.1, R8.1
- net GND: now also C23.1, C24.2, C28.1, C31.1, C46.1, C47.2, C48.1, C49.2, C58.2, CNP4.1, CNP4.13, CNP4.14, CNP4.26, IC10.1 (1A), IC10.12 (4A), IC10.13 (4B), IC10.4 (2A), IC10.7 (GND), IC10.9 (3A), IC18.3 (VSS), NF4.2, OSC1.4 (GND), R51.1, R67.1
- net at IC5.11 (CX): now also R44.1
- net at IC5.113 (DVDD3), IC5.13 (DVDD1), IC5.25 (DVDD4)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: now also C23.2, C46.2, C47.1, C48.2, C49.1, R26.1, R33.1, R34.1
- net at IC5.12 (~{HDRES}): now also IC18.1 (OUT), R51.2
- net ~{EQMD}: now reaches IC5.20 (~{EQMD})
- net ~{EYCY}: now reaches IC5.22 (~{EYCY})
- net at IC5.30 (RXLPIN): now also C34.1
- net at IC5.42 (MOD0), IC5.45 (MOD3): now also R41.2
- net MN195_ADCK# renamed ~{VSCK}
- net ~{VSCK}: now also CNP4.21, IC5.95 (~{VSCK}); no longer IC5.95 (VSCK#)
- net MN195_AGCIN: no longer names the net of IC5.28 (AGCIN)
- net MN195_AGCIN: now also IC3.18
- net MN195_AGCOUT: no longer names the net of IC5.27 (AGCOUT)
- net MN195_AGCOUT: now also IC3.17
- net MN195_HPOUT: no longer names the net of IC5.29 (HPOUT)
- net MN195_HPOUT: now also IC3.6
- net MN195_HVDD renamed MODULE_2
- net MODULE_2: now also IC3.2
- net MN195_IREF0: no longer names the net of IC5.38 (IREF0)
- net MN195_IREF0: now also R10.1
- net MN195_IREF1: no longer names the net of IC5.37 (IREF1)
- net MN195_IREF1: now also C2.1, R10.2, R11.1
- net MN195_IREF2: no longer names the net of IC5.31 (IREF2)
- net MN195_IREF2: now also C34.2
- removed net MN195_IRQ1#: IC5.67 (IRQ1#)
- removed net MN195_MTA1: IC5.92 (MTA1)
- net MN195_PLSD: no longer names the net of IC5.23 (PLSD)
- net MN195_PLSD: now also IC3.1
- net MN195_RXL: no longer names the net of IC5.32 (RXL)
- net MN195_RXL: now also IC3.3
- removed net MN195_S1: IC5.47 (S1)
- removed net MN195_S10: IC5.56 (S10)
- removed net MN195_S11: IC5.57 (S11)
- removed net MN195_S3: IC5.49 (S3)
- removed net MN195_S4: IC5.50 (S4)
- removed net MN195_S5: IC5.51 (S5)
- removed net MN195_S6: IC5.52 (S6)
- removed net MN195_S7: IC5.53 (S7)
- removed net MN195_S8: IC5.54 (S8)
- removed net MN195_S9: IC5.55 (S9)
- net MN195_SHIN: no longer names the net of IC5.26 (SHIN)
- net MN195_SHIN: now also IC3.16
- net MN195_TXLPIN: no longer names the net of IC5.36 (TXLPIN)
- net MN195_TXLPIN: now also C2.2, IC3.9, R11.2
- net MN195_TXOUT: no longer names the net of IC5.34 (TXOUT)
- net MN195_TXOUT: now also IC3.10
- removed net MN195_U1RD: IC5.63 (U1RD#)
- removed net MN195_U1SD: IC5.65 (U1SD#)
- removed net MN195_VPCK#: IC5.87 (VPCK#)
- removed net MN195_VPDA#: IC5.88 (VPDA#)
- net MN195_VREEH: no longer names the net of IC5.39 (AVDD), IC5.40 (VREFH)
- net MN195_VREEH: now also C45.2 (1), R35.2
- removed net MN195_VSDA#: IC5.96 (VSDA#)
- removed net MN195_VSEN#: IC5.98 (VSEN#)
- new net: C73.2, IC17.2 (I), R100.2
- new net: C71.1, DA1.2 (A2), R99.1
- new net: CNP4.5, IC10.2 (1B), R22.2
- new net: IC10.3 (1Y), R16.1
- new net: C58.1, D5.1 (A1), D5.2 (A2), IC18.2 (VDD), R49.2
- new net: CNP4.3, IC10.10 (3B), R27.1
- new net: C72.1, IC3.12, R99.2
- new net: C70.1, IC17.4 (O), R100.1
- new net: C70.2, DA1.1 (A1), DA1.4 (C2)
- new net: Q3.3 (C), Q4.1 (B), R1.1, R76.2, R8.2
- new net: C32.2, R76.1
- new net: NF2.1, R26.2, R33.2, R34.2
- new net: C74.1, IC17.5 (VCC), R98.1
- new net: C24.1, NF3.1, OSC1.2 (VCC)
- new net: NF1.1, R35.1
- new net: C32.1, IC3.8
- new net: IC10.8 (3Y), R19.2
- new net: OSC1.1 (OUT), R44.2
- new net: IC5.68 (~{IRQ2}), R43.2
- new net: CNP4.8, IC10.5 (2B), R23.2
- new net: IC10.6 (2Y), R17.1
- new net +5V: C28.2, CNP4.2, CNP4.25, D5.3 (C), IC10.14 (VCC), NF2.2, NF3.2, R133.1, R21.1, R3.2, R41.1, R43.1, R47.1, R48.2, R49.1, R72.1, R79.1
- new net +5V_STBY: C31.2, CNP4.12, CNP4.15
- new net AVDD: C57.2, IC3.13, NF1.2, Q4.3 (C), R1.2, R48.1, R98.2
- new net CNP4_22: CNP4.22, Q4.2 (E), R52.2
- new net CTS: CNP4.6, IC5.54 (S8)
- new net DCD: CNP4.10, IC5.52 (S6)
- new net DSR: CNP4.7, IC5.51 (S5)
- new net DTR: IC5.56 (S10), R17.2, R23.1
- new net FAX_ENABLE: IC5.48 (S2), R47.2
- new net FAX_SIGNAL: IC3.15
- new net FAX/PHONE_ENABLE: IC5.46 (S0), R21.2
- new net MODULE_11: IC3.11, IC5.92 (MTA1)
- new net MODULE_4: IC3.4, IC5.47 (S1)
- new net MODULE_5: IC3.5, IC5.50 (S4)
- new net RI: CNP4.9, IC5.53 (S7)
- new net RING: CNP4.11
- new net RING_CONTROL: IC5.49 (S3), R72.2
- new net RTS: IC5.55 (S9), R16.2, R22.1
- new net RXD: IC5.63 (~{U1RD}), R19.1, R27.2
- new net S11: IC5.57 (S11), Q3.1 (B), R133.2
- new net TXD: CNP4.4, IC5.65 (~{U1SD})
- new net VOICE_ENABLE: IC5.58 (S12), R67.2
- new net VOICE_SW_OVERWRITE: IC5.59 (S13), R79.2
- new net ~{IRQ1}: CNP4.20, IC5.67 (~{IRQ1}), R3.1
- new net ~{VPCK}: CNP4.18, IC5.87 (~{VPCK})
- new net ~{VPDA}: CNP4.19, IC5.88 (~{VPDA})
- new net ~{VSDA}: CNP4.17, IC5.96 (~{VSDA})
- new net ~{VSEN}: CNP4.16, IC5.98 (~{VSEN})
- no-connect marks 39 -> 32
Other:
- added sheet Front End (fe.kicad_sch)
- added sheet RAM and ROM (ramrom.kicad_sch)
- note added: "Speech network for FAX"
- note added: "or 2E00"
- company: Recreated by: Ahmad Byagowi -> (none)
- title: PC110 Internal Modem Module -> DVYGA1669-4 : IBM PalmTop PC110 FAX/Modem module
