File: PCB/Modem/Modem.kicad_pcb (KiCad board)
At the start: 6 copper layers, 64.6 x 58.9 mm, 212 parts, among them IC10 AT32 433, IC11 EN29F040A, IC12 KM681000BLT-7 (I-Reverse), IC13 EA, IC14 E4, IC15 8206 5877, IC16 E3, IC17 EA, IC18 3L01, IC2 EA, IC3 Line-Module, IC4 E5, IC5 MN195, IC6 54, IC7 EA, IC8 TA31033F, IC9 EA, Q1 CQ, Q2 DA QU, Q3 123, Q4 CQ, Q7 SOT-323_SC-70, Q9 HP, SW2 SW_modem, T1 IsoTransformer

Commit message: cleanup modem schematic
Parts:
- C1, C4, C54: value 330nF -> 0.33u
- C12, C45: value 47uF 16v -> 47u
- C13: value 822J -> 22u
- C15, C23, C32: value 1.2uF -> 1u
- C2, C34: value 1nF -> 1000p
- C24, C31, C37: value 230nF -> 0.22u
- C26: value 10nF -> 0.01u
- C28: value 8.1uF -> 10u
- C29, C30: value 1.5uF -> 1u
- C3: value 30nF -> 0.33u
- C38: value 2.2uF -> 2700p
- C39: value 100nF -> 0.1u
- C40: value 16nF -> 0.022u
- C41: value 1uF -> 1000p
- C42, C51: value 1.2nF -> 1u
- C43: value 1uF -> 1u
- C46, C47: value 24nF -> 0.022u
- C48: value 25nF -> 0.022u
- C49: renamed from C39; value 25nF -> 0.022u
- C5: value 250nF -> 0.22u
- C52: value 330nF -> 0.22u
- C53: renamed from C56; value 1.6nF -> 1500p
- C55: renamed from C2; value 1.2uF -> 1u
- C56: value 470nF -> 0.33u
- C57: value 6.8uF -> 8.2u
- C58, C74: value 220nF -> 0.22u
- C59, C60: value 280nF -> 0.33u
- C62: value 280nF -> 0.22u
- C70, C72: value 1.8uF -> 1u
- C71: value 1.3uF -> 1u
- C73: value 100pF -> 100p
- CNP1: value Line_Connector -> CRS5001-0201
- CNP2: value modem_heaset_jack -> HSJ1102-01-510
- CNP3: value JST_8_headset_connector -> 52271-0890
- CNP4: value Modem-Connector -> 8-176757-6
- CNP5: value JST_2_modem_spkr -> DF13-2P-1.25H
- D1, D7, D9: value TO-269AA -> S1ZB60
- D10: value 152 -> 02DZ15
- D2: value 1N4148 -> RLZ12A
- D3, D4, D8: value 5 -> 1SV203
- D5: value 3D -> RB715F
- D6: value 30H -> MAZ33000H
- DA1: value M1T -> MA724
- IC10: value AT32 433 -> TC74ACT32FT
- IC11: value EN29F040A -> MBM29F040A-12
- IC12: value KM681000BLT-7 (I-Reverse) -> KM681000BLT-7
- IC13, IC17, IC2, IC7, IC9: value EA -> TC7S14FU
- IC14: value E4 -> TC7S32FU
- IC15: value 8206 5877 -> BA8206F
- IC16: value E3 -> TC7S02FU
- IC18: value 3L01 -> R3111N331C
- IC3: value Line-Module -> ~
- IC4: value E5 -> TC7S04FU
- IC5: value MN195 -> MN195001MFM-6
- IC6: value 54 -> TC7S32FU
- L1, L2, L4: value 1.2uH -> 1.5u
- L3, L5: value 1.8uH -> 1.5u
- NF1: value 300nH -> 330n
- NF2: value 4.7nH -> 560n
- NF4: value 4.7nH -> 330n
- OSC1: value 41.472 -> 41.472MHz
- Q1, Q4: value CQ -> 2SC4097-Q
- Q2: value DA QU -> 2SD1664-Q
- Q3: value 123 -> DTC143ZUA
- Q6: renamed from Q9; value HP -> 2SA1577-P
- Q7: value SOT-323_SC-70 -> DTC143ZUA
- R10, R11, R68: value 38k -> 39k
- R15: value 330k -> 270k
- R16, R17, R19: value 10k -> 100
- R22, R23, R27: value DNP -> ~
- R25: value 500k -> 510k
- R53: value 11k -> 10k
- R59: value 2.2k -> 22k
- R70, R71: value 1k -> 1.2k
- R77: value 270k -> 330k
- R8: value 22k -> 12k
- RL1: value RL -> AQW210S
- SW2: value SW_modem -> ~
- T1: value IsoTransformer -> ~
- VA1: value R_2512_6332Metric -> ERZCF2MK361
- renumbered R124 to R128, R68 to R69, R9 to R7, R72 to R79, R7 to R9
Connections:
- net C32_1 renamed Net-(C32-Pad1)
- net C32_2 renamed Net-(C32-Pad2)
- net C39_1 renamed Net-(C39-Pad1)
- net C40_2 renamed Net-(C40-Pad2)
- net C51_1 renamed Net-(C51-Pad1)
- net C70_1 renamed Net-(IC17A-O)
- net C70_2 renamed Net-(DA1A-A1)
- net C72_1 renamed Net-(C72-Pad1)
- net C74_1 renamed Net-(IC17B-VCC)
- net CNP2_2 renamed Net-(CNP2-Pad2)
- net CNP2_3 renamed Net-(CNP2-Pad3)
- net CNP3_1 renamed Net-(CNP2-Pad4)
- net CNP3_5 renamed Net-(CNP3-Pad5)
- net CNP5_1 renamed Net-(CNP5-Pad1)
- net D1_1 renamed Net-(D1-+)
- net D1_2 renamed Net-(C15-Pad1)
- net D2_2 renamed Net-(D2-A)
- net D4_1 renamed Net-(D4-C)
- net D7_1 renamed Net-(D6-C)
- net D7_3 renamed Net-(C59-Pad1)
- net DA1_2 renamed Net-(DA1B-C2)
- net FDC_CTS1# renamed Net-(IC10B-2B)
- net FDC_DCD1_PC110 renamed TXD
- net FDC_DIR1#_PC110 renamed CTS
- net FDC_DSR1_PC110 renamed DSR
- net FDC_RI1_PC110 renamed Net-(IC10A-1B)
- net FDC_RTS1#_PC110 renamed RI
- net FDC_RXD1_PC110 renamed DCD
- net FDC_TXD1_PC110 renamed RING
- net IC10_6 renamed Net-(IC10B-2Y)
- net IC10_8 renamed Net-(IC10C-3Y)
- net IC12_3 renamed Net-(IC12-~{CS1})
- net IC13_2 renamed Net-(IC13A-I)
- net IC13_4 renamed Net-(D8-C)
- net IC14_1 renamed Net-(IC14A-I0)
- net IC14_4 renamed Net-(IC14A-O)
- net IC15_2 renamed Net-(IC15-RSL)
- net IC15_3 renamed Net-(IC15-LFI)
- net IC15_4 renamed Net-(IC15-LFO)
- net IC15_6 renamed Net-(IC15-HFO)
- net IC15_7 renamed Net-(IC15-HFI)
- net IC15_8 renamed Net-(IC15-OUT)
- net IC16_1 renamed Net-(D3-C)
- net IC16_4 renamed Net-(IC14A-I1)
- net IC17_2 renamed Net-(IC17A-I)
- net IC18_2 renamed Net-(D5-A1)
- net IC3_15 renamed FAX_SIGNAL
- net IC6_2 renamed Net-(IC4A-O)
- net IC7_4 renamed Net-(IC7A-O)
- net IC8_10 renamed Net-(IC8-TPI_2)
- net IC8_11 renamed Net-(IC8-TPI_1)
- net IC8_12 renamed Net-(IC8-PADC)
- net IC8_13 renamed Net-(IC8-RPI_1)
- net IC8_14 renamed Net-(IC8-RPO)
- net IC8_15 renamed Net-(C13-2)
- net IC8_16 renamed Net-(C12-1)
- net IC8_3 renamed Net-(IC8-TOO)
- net IC8_5 renamed Net-(IC8-MFI)
- net IC8_7 renamed Net-(IC8-REF)
- net IC8_9 renamed Net-(IC8-TPO)
- net IC9_2 renamed Net-(IC9A-I)
- net IREF2 renamed Net-(IC5A-IREF2)
- net L1_1 renamed Net-(D1--)
- net L1_2 renamed Net-(L2-Pad2)
- net L3_1 renamed Net-(C42-Pad1)
- net L3_2 renamed Net-(CNP2-Pad1)
- net L4_1 renamed Net-(L4-Pad1)
- net L5_2 renamed Net-(CNP2-Pad5)
- net MN192_S11_BUF renamed CNP4_22
- net MN195_A0 renamed Net-(IC5B-A0)
- net MN195_A1 renamed Net-(IC5B-A1)
- net MN195_A10 renamed Net-(IC5B-A10)
- net MN195_A11 renamed Net-(IC5B-A11)
- net MN195_A12 renamed Net-(IC5B-A12)
- net MN195_A13 renamed Net-(IC5B-A13)
- net MN195_A14 renamed Net-(IC5B-A14)
- net MN195_A15 renamed Net-(IC5B-A15)
- net MN195_A16 renamed Net-(IC5B-A16)
- net MN195_A17 renamed Net-(IC5B-A17)
- net MN195_A18 renamed Net-(IC5B-A18)
- net MN195_A2 renamed Net-(IC5B-A2)
- net MN195_A3 renamed Net-(IC5B-A3)
- net MN195_A4 renamed Net-(IC5B-A4)
- net MN195_A5 renamed Net-(IC5B-A5)
- net MN195_A6 renamed Net-(IC5B-A6)
- net MN195_A7 renamed Net-(IC5B-A7)
- net MN195_A8 renamed Net-(IC5B-A8)
- net MN195_A9 renamed Net-(IC5B-A9)
- net MN195_ADCK# renamed ~{VSCK}
- net MN195_AGCIN renamed Net-(IC5A-AGCIN)
- net MN195_AGCOUT renamed Net-(IC5A-AGCOUT)
- net MN195_CX renamed Net-(IC5A-CX)
- net MN195_DVDD1 renamed Net-(IC5A-DVDD1)
- net MN195_EQMD# renamed ~{EQMD}
- net MN195_EYCY# renamed ~{EYCY}
- net MN195_HDRES# renamed Net-(IC18-OUT)
- net MN195_HPOUT renamed Net-(IC5A-HPOUT)
- net MN195_HVDD renamed MODULE_2
- net MN195_IREF0 renamed Net-(IC5A-IREF0)
- net MN195_IREF1 renamed Net-(IC5A-IREF1)
- net MN195_IRQ1# renamed ~{IRQ1}
- net MN195_IRQ2# renamed Net-(IC5C-~{IRQ2})
- net MN195_MD0 renamed Net-(IC5B-MD0)
- net MN195_MD1 renamed Net-(IC5B-MD1)
- net MN195_MD2 renamed Net-(IC5B-MD2)
- net MN195_MD3 renamed Net-(IC5B-MD3)
- net MN195_MD4 renamed Net-(IC5B-MD4)
- net MN195_MD5 renamed Net-(IC5B-MD5)
- net MN195_MD6 renamed Net-(IC5B-MD6)
- net MN195_MD7 renamed Net-(IC5B-MD7)
- net MN195_MOD1,3 renamed Net-(IC5A-MOD0)
- net MN195_MTA1 renamed MODULE_11
- net MN195_PLSD renamed Net-(IC5A-PLSD)
- net MN195_RD# renamed Net-(IC5B-~{RD})
- net MN195_RXL renamed Net-(IC5A-RXL)
- net MN195_S0 renamed FAX/PHONE_ENABLE
- net MN195_S1 renamed MODULE_4
- net MN195_S10 renamed DTR
- net MN195_S11 renamed S11
- net MN195_S12 renamed VOICE_ENABLE
- net MN195_S13 renamed VOICE_SW_OVERWRITE
- net MN195_S2 renamed FAX_ENABLE
- net MN195_S3 renamed RING_CONTROL
- net MN195_S4 renamed MODULE_5
- net MN195_S9 renamed RTS
- net MN195_SHIN renamed Net-(IC5A-SHIN)
- net MN195_TXLPIN renamed Net-(IC5A-TXLPIN)
- net MN195_TXOUT renamed Net-(IC5A-TXOUT)
- net MN195_U1RD# renamed RXD
- net MN195_U1RD#_R renamed Net-(IC10C-3B)
- net MN195_UC0# renamed Net-(IC5B-~{UC0})
- net MN195_UC1 renamed Net-(IC5B-~{UC1})
- net MN195_VPCK# renamed ~{VPCK}
- net MN195_VPDA# renamed ~{VPDA}
- net MN195_VREEH renamed Net-(C45-1)
- net MN195_VSDA# renamed ~{VSDA}
- net MN195_VSEN# renamed ~{VSEN}
- net MN195_WR# renamed Net-(IC5B-~{WR})
- net NF1_1 renamed Net-(NF1-Pad1)
- net NF2_1 renamed Net-(NF2-Pad1)
- net OSC1_1 renamed Net-(OSC1-OUT)
- net OSC1_2 renamed Net-(OSC1-VCC)
- net PC2_1 renamed Net-(PC2-A)
- net PNET1 renamed AVDD
- net PNET4 renamed AGND
- net Pluto_Enabled_PNET5 renamed +5V_STBY
- net Q3_3 renamed Net-(Q3-C)
- net Q7_1 renamed Net-(Q7-B)
- net Q9_1 renamed Net-(Q6-B)
- net R12_2 renamed Net-(C62-Pad2)
- net R16_1 renamed Net-(IC10A-1Y)
- net R24_2 renamed Net-(CNP3-Pad7)
- net R54_1 renamed Net-(D10-C)
- net R54_2 renamed Net-(C26-Pad2)
- net R55_1 renamed Net-(Q6-C)
- net R56_2 renamed Net-(C12-2)
- net R57_2 renamed Net-(C26-Pad1)
- net R61_2 renamed Net-(C56-Pad1)
- net R65_2 renamed Net-(C13-1)
- net R73_2 renamed Net-(IC2A-I)
- net R75_1 renamed Net-(C59-Pad2)
- net R82_2 renamed Net-(R61-Pad1)
- net RL1_2 renamed Net-(R46-Pad2)
- net RL1_3 renamed Net-(R18-Pad2)
- net RL1_4 renamed Net-(IC6A-O)
- net RL1_5 renamed Net-(C1-Pad1)
- net RL1_7 renamed Net-(D9-AC-Pad3)
- net T1_4 renamed Net-(C1-Pad2)
- net TEL_GND renamed Net-(CNP1-PAD-Pad2)
- net TEL_Line renamed Net-(CNP1-Pad1)
- net TLP124_4 renamed Net-(PC2-E)
- C28 pad 2: VCC_PC110 -> +5V
- C29 pad 2: VCC_PC110 -> +5V
- C30 pad 1: VCC_PC110 -> +5V
- C34 pad 1: C34_1 -> Net-(IC5A-RXLPIN)
- C52 pad 2: C52_2 -> Net-(D6-A)
- C53 pad 1: C52_2 -> Net-(D6-A)
- C54 pad 1: C52_2 -> Net-(D6-A)
- CNP3 pad 6: CNP5_2 -> Net-(D6-A)
- CNP3 pad MP: CNP3_MP1 -> unconnected-(CNP3-PadMP)
- CNP4 pad 2: VCC_PC110 -> +5V
- CNP4 pad 23: J13_41_PC110 -> unconnected-(CNP4-Pad23)
- CNP4 pad 24: J13_42_PC110 -> unconnected-(CNP4-Pad24)
- CNP4 pad 25: VCC_PC110 -> +5V
- CNP5 pad 2: CNP5_2 -> Net-(D6-A)
- CNP5 pad MP: CNP5_MP1 -> unconnected-(CNP5-PadMP)
- D5 pad 3: VCC_PC110 -> +5V
- D6 pad 1: C52_2 -> Net-(D6-A)
- D6 pad 2: D6_2 -> (no net)
- D7 pad 2: C52_2 -> Net-(D6-A)
- IC10 pad 11: IC10_11 -> unconnected-(IC10D-4Y-Pad11)
- IC10 pad 14: VCC_PC110 -> +5V
- IC11 pad 1: 29F_OE# -> /RAM and ROM/MEM_A11
- IC11 pad 10: 29F_DQ2 -> /RAM and ROM/MEM_A16
- IC11 pad 11: 29F_DQ1 -> /RAM and ROM/MEM_A15
- IC11 pad 12: 29F_DQ0 -> /RAM and ROM/MEM_A12
- IC11 pad 13: 29F_A0 -> /RAM and ROM/MEM_A7
- IC11 pad 14: 29F_A1 -> /RAM and ROM/MEM_A6
- IC11 pad 15: 29F_A2 -> /RAM and ROM/MEM_A5
- IC11 pad 16: 29F_A3 -> /RAM and ROM/MEM_A4
- IC11 pad 17: 29F_A4 -> /RAM and ROM/MEM_A3
- IC11 pad 18: 29F_A5 -> /RAM and ROM/MEM_A2
- IC11 pad 19: 29F_A6 -> /RAM and ROM/MEM_A1
- IC11 pad 2: 29F_A10 -> /RAM and ROM/MEM_A9
- IC11 pad 20: 29FA7 -> /RAM and ROM/MEM_A0
- IC11 pad 21: 29F_A12 -> /RAM and ROM/MEM_D0
- IC11 pad 22: 29F_A15 -> /RAM and ROM/MEM_D1
- IC11 pad 23: 29F_A16 -> /RAM and ROM/MEM_D2
- IC11 pad 24: 29F_A18 -> GND
- IC11 pad 25: VCC_PC110 -> /RAM and ROM/MEM_D3
- IC11 pad 26: 29F_WE# -> /RAM and ROM/MEM_D4
- IC11 pad 27: 29F_A17 -> /RAM and ROM/MEM_D5
- IC11 pad 28: 29F_A14 -> /RAM and ROM/MEM_D6
- IC11 pad 29: 29F_A13 -> /RAM and ROM/MEM_D7
- IC11 pad 3: 29F_CE# -> /RAM and ROM/MEM_A8
- IC11 pad 30: 29F_A8 -> Net-(IC11-~{CE})
- IC11 pad 31: 29F_A9 -> /RAM and ROM/MEM_A10
- IC11 pad 32: 29F_A11 -> Net-(IC11-~{OE})
- IC11 pad 4: 29F_DQ7 -> /RAM and ROM/MEM_A13
- IC11 pad 5: 29F_DQ6 -> /RAM and ROM/MEM_A14
- IC11 pad 6: 29F_DQ5 -> /RAM and ROM/MEM_A17
- IC11 pad 7: 29F_DQ4 -> Net-(IC11-~{WE})
- IC11 pad 8: 29F_DQ3 -> +5V
- IC11 pad 9: GND -> /RAM and ROM/MEM_A18
- IC12 pad 1: 29F_A11 -> /RAM and ROM/MEM_A11
- IC12 pad 10: 29F_A16 -> /RAM and ROM/MEM_A16
- IC12 pad 11: 29F_A14 -> /RAM and ROM/MEM_A14
- IC12 pad 12: 29F_A12 -> /RAM and ROM/MEM_A12
- IC12 pad 13: 29FA7 -> /RAM and ROM/MEM_A7
- IC12 pad 14: 29F_A6 -> /RAM and ROM/MEM_A6
- IC12 pad 15: 29F_A5 -> /RAM and ROM/MEM_A5
- IC12 pad 16: 29F_A4 -> /RAM and ROM/MEM_A4
- IC12 pad 17: 29F_A3 -> /RAM and ROM/MEM_A3
- IC12 pad 18: 29F_A2 -> /RAM and ROM/MEM_A2
- IC12 pad 19: 29F_A1 -> /RAM and ROM/MEM_A1
- IC12 pad 2: 29F_A9 -> /RAM and ROM/MEM_A9
- IC12 pad 20: 29F_A0 -> /RAM and ROM/MEM_A0
- IC12 pad 21: 29F_DQ0 -> /RAM and ROM/MEM_D0
- IC12 pad 22: 29F_DQ1 -> /RAM and ROM/MEM_D1
- IC12 pad 23: 29F_DQ2 -> /RAM and ROM/MEM_D2
- IC12 pad 25: 29F_DQ3 -> /RAM and ROM/MEM_D3
- IC12 pad 26: 29F_DQ4 -> /RAM and ROM/MEM_D4
- IC12 pad 27: 29F_DQ5 -> /RAM and ROM/MEM_D5
- IC12 pad 28: 29F_DQ6 -> /RAM and ROM/MEM_D6
- IC12 pad 29: 29F_DQ7 -> /RAM and ROM/MEM_D7
- IC12 pad 3: 29F_A8 -> /RAM and ROM/MEM_A8
- IC12 pad 31: 29F_A10 -> /RAM and ROM/MEM_A10
- IC12 pad 32: 29F_OE# -> Net-(IC11-~{OE})
- IC12 pad 4: 29F_A13 -> /RAM and ROM/MEM_A13
- IC12 pad 5: 29F_WE# -> Net-(IC11-~{WE})
- IC12 pad 6: VCC_PC110 -> +5V
- IC12 pad 7: 29F_A15 -> /RAM and ROM/MEM_A15
- IC12 pad 8: VCC_PC110 -> +5V
- IC12 pad 9: KM68_NC -> (no net)
- IC13 pad 1: IC13_1 -> (no net)
- IC15 pad 5: C52_2 -> Net-(D6-A)
- IC17 pad 1: IC17_1 -> (no net)
- IC18 pad 4: IC18_4 -> (no net)
- IC18 pad 5: IC18_5 -> (no net)
- IC2 pad 1: IC2_1 -> (no net)
- IC4 pad 1: IC4_1 -> (no net)
- IC4 pad 5: VCC_PC110 -> +5V
- IC5 pad 101: MN195_UC2 -> unconnected-(IC5B-~{UC2}-Pad101)
- IC5 pad 102: MN195_UC3 -> unconnected-(IC5B-~{UC3}-Pad102)
- IC5 pad 103: MN195_A23 -> unconnected-(IC5B-A23-Pad103)
- IC5 pad 104: MN195_A22 -> unconnected-(IC5B-A22-Pad104)
- IC5 pad 105: MN195_A21 -> unconnected-(IC5B-A21-Pad105)
- IC5 pad 106: MN195_A20 -> unconnected-(IC5B-A20-Pad106)
- IC5 pad 107: MN195_A19 -> unconnected-(IC5B-A19-Pad107)
- IC5 pad 17: MN195_RNW -> unconnected-(IC5B-R/W-Pad17)
- IC5 pad 18: MN195_BA -> unconnected-(IC5A-BA-Pad18)
- IC5 pad 30: MN195_RXLPIN -> Net-(IC5A-RXLPIN)
- IC5 pad 60: MN195_S14 -> unconnected-(IC5C-S14-Pad60)
- IC5 pad 61: MN195_S15 -> unconnected-(IC5C-S15-Pad61)
- IC5 pad 62: MN195_U1ST# -> unconnected-(IC5C-~{U1ST}-Pad62)
- IC5 pad 64: MN195_U1RCK -> unconnected-(IC5C-~{U1RCK}-Pad64)
- IC5 pad 66: MN195_U1TCK# -> unconnected-(IC5C-~{U1TCK}-Pad66)
- IC5 pad 69: MN195_IRQ3# -> unconnected-(IC5C-~{IRQ3}-Pad69)
- IC5 pad 70: MN195_IRQ4# -> unconnected-(IC5C-~{IRQ4}-Pad70)
- IC5 pad 71: MN195_U2ST# -> unconnected-(IC5C-~{U2ST}-Pad71)
- IC5 pad 72: MN195_U2RD# -> unconnected-(IC5C-~{U2RD}-Pad72)
- IC5 pad 73: MN195_U2RCK# -> unconnected-(IC5C-~{U2RCK}-Pad73)
- IC5 pad 74: MN195_U2SD# -> unconnected-(IC5C-~{U2SD}-Pad74)
- IC5 pad 75: MN195_U2TCK# -> unconnected-(IC5C-~{U2TCK}-Pad75)
- IC5 pad 78: MN195_MTB4 -> unconnected-(IC5C-MTB4-Pad78)
- IC5 pad 79: MN195_MTB3 -> unconnected-(IC5C-MTB3-Pad79)
- IC5 pad 80: MN195_MTB2 -> unconnected-(IC5C-MTB2-Pad80)
- IC5 pad 81: MN195_MTB1 -> unconnected-(IC5C-MTB1-Pad81)
- IC5 pad 82: MN195_SH4# -> unconnected-(IC5C-~{SH4}-Pad82)
- IC5 pad 83: MN195_SH3# -> unconnected-(IC5C-~{SH3}-Pad83)
- IC5 pad 84: MN195_SH2# -> unconnected-(IC5C-~{SH2}-Pad84)
- IC5 pad 85: MN195_SH1# -> unconnected-(IC5C-~{SH1}-Pad85)
- IC5 pad 86: MN195_VPST -> unconnected-(IC5C-VPST-Pad86)
- IC5 pad 89: MN195_MTA4 -> unconnected-(IC5C-MTA4-Pad89)
- IC5 pad 9: MN195_SYNCA -> unconnected-(IC5A-SYNCA-Pad9)
- IC5 pad 90: MN195_MTA3 -> unconnected-(IC5C-MTA3-Pad90)
- IC5 pad 91: MN195_MTA2 -> unconnected-(IC5C-MTA2-Pad91)
- IC5 pad 93: MN195_MOT -> unconnected-(IC5C-MOT-Pad93)
- IC5 pad 94: MN195_V8CK# -> unconnected-(IC5C-~{V8CK}-Pad94)
- IC5 pad 97: MN195_VIR# -> unconnected-(IC5C-~{VIR}-Pad97)
- IC6 pad 5: VCC_PC110 -> +5V
- IC7 pad 1: IC7_1 -> (no net)
- IC8 pad 2: IC8_2 -> Net-(IC8-TOI)
- IC8 pad 4: IC8_4 -> unconnected-(IC8-AC_BIAS-Pad4)
- IC8 pad 6: IC8_6 -> unconnected-(IC8-MUTE-Pad6)
- IC9 pad 1: IC9_1 -> (no net)
- NF2 pad 2: VCC_PC110 -> +5V
- NF3 pad 2: VCC_PC110 -> +5V
- OSC1 pad 3: OSC1_3 -> (no net)
- PC2 pad 3: C52_2 -> Net-(D6-A)
- Q1 pad 2: Q2_1 -> Net-(Q1-E)
- Q2 pad 1: Q2_1 -> Net-(Q1-E)
- Q2 pad 3: Q2_1 -> Net-(Q2-E)
- R101 pad 1: 29F_CE# -> Net-(IC11-~{CE})
- R102 pad 1: 29F_A18 -> /RAM and ROM/MEM_A18
- R103 pad 1: 29F_A16 -> /RAM and ROM/MEM_A16
- R104 pad 1: 29F_A14 -> /RAM and ROM/MEM_A14
- R105 pad 1: 29F_A12 -> /RAM and ROM/MEM_A12
- R106 pad 1: 29F_A10 -> /RAM and ROM/MEM_A10
- R107 pad 1: 29F_A8 -> /RAM and ROM/MEM_A8
- R108 pad 1: 29F_A6 -> /RAM and ROM/MEM_A6
- R109 pad 1: 29F_A4 -> /RAM and ROM/MEM_A4
- R110 pad 1: 29F_A2 -> /RAM and ROM/MEM_A2
- R111 pad 1: 29F_A0 -> /RAM and ROM/MEM_A0
- R114 pad 1: 29F_A17 -> /RAM and ROM/MEM_A17
- R115 pad 1: 29F_A15 -> /RAM and ROM/MEM_A15
- R116 pad 1: 29F_A13 -> /RAM and ROM/MEM_A13
- R117 pad 1: 29F_A11 -> /RAM and ROM/MEM_A11
- R118 pad 1: 29F_A9 -> /RAM and ROM/MEM_A9
- R119 pad 1: 29FA7 -> /RAM and ROM/MEM_A7
- R120 pad 1: 29F_A5 -> /RAM and ROM/MEM_A5
- R121 pad 1: 29F_A3 -> /RAM and ROM/MEM_A3
- R122 pad 1: 29F_A1 -> /RAM and ROM/MEM_A1
- R123 pad 1: 29F_OE# -> Net-(IC11-~{OE})
- R124 pad 1: 29F_WE# -> Net-(IC11-~{WE})
- R125 pad 1: 29F_DQ0 -> /RAM and ROM/MEM_D0
- R126 pad 1: 29F_DQ1 -> /RAM and ROM/MEM_D1
- R127 pad 1: 29F_DQ2 -> /RAM and ROM/MEM_D2
- R128 pad 1: 29F_DQ3 -> /RAM and ROM/MEM_D3
- R129 pad 1: 29F_DQ4 -> /RAM and ROM/MEM_D4
- R130 pad 1: 29F_DQ5 -> /RAM and ROM/MEM_D5
- R131 pad 1: 29F_DQ6 -> /RAM and ROM/MEM_D6
- R132 pad 1: 29F_DQ7 -> /RAM and ROM/MEM_D7
- R133 pad 1: VCC_PC110 -> +5V
- R18 pad 1: VCC_PC110 -> +5V
- R21 pad 1: VCC_PC110 -> +5V
- R28 pad 1: VCC_PC110 -> +5V
- R28 pad 2: 29F_DQ0 -> /RAM and ROM/MEM_D0
- R29 pad 1: VCC_PC110 -> +5V
- R29 pad 2: 29F_DQ1 -> /RAM and ROM/MEM_D1
- R3 pad 2: VCC_PC110 -> +5V
- R30 pad 1: VCC_PC110 -> +5V
- R30 pad 2: 29F_DQ2 -> /RAM and ROM/MEM_D2
- R31 pad 1: VCC_PC110 -> +5V
- R31 pad 2: 29F_DQ3 -> /RAM and ROM/MEM_D3
- R32 pad 1: VCC_PC110 -> +5V
- R32 pad 2: 29F_DQ4 -> /RAM and ROM/MEM_D4
- R36 pad 1: VCC_PC110 -> +5V
- R36 pad 2: 29F_DQ5 -> /RAM and ROM/MEM_D5
- R37 pad 1: VCC_PC110 -> +5V
- R37 pad 2: 29F_DQ6 -> /RAM and ROM/MEM_D6
- R38 pad 1: VCC_PC110 -> +5V
- R38 pad 2: 29F_DQ7 -> /RAM and ROM/MEM_D7
- R41 pad 1: VCC_PC110 -> +5V
- R42 pad 2: C52_2 -> Net-(D6-A)
- R43 pad 1: VCC_PC110 -> +5V
- R47 pad 1: VCC_PC110 -> +5V
- R48 pad 2: VCC_PC110 -> +5V
- R49 pad 1: VCC_PC110 -> +5V
- R5 pad 1: R6_2 -> Net-(IC8-TOI)
- R6 pad 2: R6_2 -> Net-(IC8-TOI)
- R72 pad 1: VCC_PC110 -> +5V
- R79 pad 1: VCC_PC110 -> +5V
- R82 pad 1: C52_2 -> Net-(D6-A)
- R9 pad 1: Q2_1 -> Net-(Q2-E)
- R90 pad 1: VCC_PC110 -> +5V
- SW2 pad 1: SW2_1 -> unconnected-(SW2-Pad1)
- SW2 pad MP: SW2_MP4 -> unconnected-(SW2-PadMP)_1
Routing:
- net VCC_PC110: track 164.8 -> 0.00 mm, vias 13 -> 0
- net +5V: track 0.00 -> 164.7 mm, vias 0 -> 13
- net Net-(D6-A): track 0.00 -> 111.4 mm, vias 0 -> 4
- net C52_2: track 91.8 -> 0.00 mm, vias 4 -> 0
- net 29F_DQ6: track 54.5 -> 0.00 mm, vias 3 -> 0
- net /RAM and ROM/MEM_D6: track 0.00 -> 54.5 mm, vias 0 -> 3
- net 29F_DQ5: track 52.9 -> 0.00 mm, vias 3 -> 0
- net /RAM and ROM/MEM_D5: track 0.00 -> 52.9 mm, vias 0 -> 3
- net 29F_DQ4: track 50.3 -> 0.00 mm, vias 3 -> 0
- net /RAM and ROM/MEM_D4: track 0.00 -> 50.3 mm, vias 0 -> 3
- net 29F_A0: track 49.8 -> 0.00 mm, vias 3 -> 0
- net /RAM and ROM/MEM_A0: track 0.00 -> 49.8 mm, vias 0 -> 3
- net 29F_A3: track 49.4 -> 0.00 mm, vias 4 -> 0
- net /RAM and ROM/MEM_A3: track 0.00 -> 49.4 mm, vias 0 -> 4
- net 29F_A1: track 47.9 -> 0.00 mm, vias 3 -> 0
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- added copper zone on B.Cu, net (none)
- added copper zone on In3.Cu, net +5V
- removed copper zone on B.Cu, net VCC_PC110
- removed copper zone on In3.Cu, net VCC_PC110

Commit message: assign bus label and fix copper zone net
Routing:
- added copper zone on B.Cu, net +5V
- removed copper zone on B.Cu, net (none)
