File: PCB/Modem/ramrom.kicad_sch (KiCad schematic)
At the start: 44 parts, among them IC11 MBM29F040A-12, IC12 KM681000BLT-7, IC5 MN195001MFM-6

Commit message: assign bus label and fix copper zone net
Changed lines of the file:
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@@
+		)
+	)
+	(label "MEM_D[0..7]"
+		(at 91.44 53.34 0)
+		(effects
+			(font
+				(size 1.27 1.27)
+			)
+			(justify left bottom)
 		)
 	)
@@
 		)
 	)
+	(label "MEM_A[0..18]"
+		(at 33.02 58.42 0)
+		(effects
+			(font
+				(size 1.27 1.27)
+			)
+			(justify left bottom)
+		)
+	)
